Commit message: Jetson sim bring-up: launch fixes, plug layout, partial native run
bin/setup_linux.sh  — fix two bugs surfaced bringing this up on a real
  Jetson Orin NX (Yahboom) with Ubuntu 22.04 + JetPack 6.x:
    * ros-humble-ros-gzharmonic doesn't exist — fall back to the
      ros-humble-ros-gz-sim subpackages that ARE installed.
    * ROS 2 setup.bash trips set -u with unbound vars; wrap source
      in set +u/-u.

Sim/.../gem_sim/launch/sim_full.launch.py:
    * Wrap xacro Command output in ParameterValue(value_type=str) so
      ROS 2 launch doesn't try to YAML-parse the URDF.
    * Render URDF to /tmp via OpaqueFunction and spawn with -file
      instead of -topic (Humble RSP doesn't publish /robot_description
      topic by default).
    * Flatten nested-list bug in PathJoinSubstitution by computing
      world path inside an OpaqueFunction.
    * Add `headless` launch arg → passes -s to gz/ign so the sim runs
      server-only on a display-less Jetson over SSH.

Sim/.../gem_sim/urdf/gem_e4_robot.urdf.xacro:
    * Remove the stub-fallback comment block. Xacro processing of the
      ${...} substitutions inside the comment apparently confused
      Gazebo's URDF parser into double-counting base_link.
    * (Earlier commit) renamed our IMU link imu_link → vn100_link to
      avoid collision with the upstream gem-simulator's imu_link.

Hardware/JETSON_PLUG_LAYOUT.md (new) — concrete port-by-port guide for
  what to plug into the Yahboom carrier in Phase 0 (gamepad, CANable
  or direct CAN via 40-pin header, Ethernet, USB, DC barrel) and
  Phase 1+ (sensors). Notes that the kernel-level can0 interface is
  already enabled — you may not need a CANable USB dongle at all.

Status on Jetson at end of session:
  ✓ Internet (Mac NAT shim, GruberSandbox out of range)
  ✓ Repo synced, 9 packages built clean
  ✓ Gazebo headless server + sim_dbw_bridge run
  ✓ All canonical ROS topics declared (sensors, /cmd_vel, /vehicle/*)
  🟡 Cart doesn't spawn into FAU breezeway world: SDF 1.10 (Harmonic)
     vs Fortress (1.9) mismatch + URDF→SDF fixed-joint reduction
     duplicates upstream gem-simulator base_link. Path forward is
     installing Harmonic-paired ros-gz packages (not in Yahboom's
     stock image) — deferred to Phase 2 per master plan.

Co-Authored-By: Claude Opus 4.7 (1M context) <noreply@anthropic.com>

File: Sim/Cartagena_GEM_E4_workspace/ros2_ws/src/gem_sim/urdf/gem_e4_robot.urdf.xacro (robot description, xacro)
@@ -21,37 +21,9 @@
   <!-- ============ Step 1: load canonical parameters ============ -->
   <xacro:include filename="$(find gem_sim)/urdf/cart_parameters.xacro"/>
-  <!-- ============ Step 2: include upstream chassis URDF ============
-       The upstream GEM-Illinois URDF defines: base_footprint, base_link,
-       chair_link, door_link, front_rack_link, the four wheels (front_left,
-       front_right, rear_left, rear_right), and the steering hinges.
-       If you want to bypass the upstream and use a minimal stub for sim-only
-       testing, comment out this include and uncomment the stub below.
-  -->
+  <!-- Step 2: include upstream chassis URDF.
+       The GEM-Illinois URDF defines base_footprint, base_link, the four
+       wheels, steering hinges, etc. We attach our sensor stack on top. -->
   <xacro:include filename="$(find gem_description)/urdf/e4/gem_e4.urdf.xacro"/>
-  <!-- Stub fallback — uncomment to test without the upstream package
-  <link name="base_footprint"/>
-  <link name="base_link">
-    <visual>
-      <origin xyz="0 0 ${VEHICLE_HEIGHT_M / 2}" rpy="0 0 0"/>
-      <geometry><box size="${VEHICLE_LENGTH_M} ${VEHICLE_WIDTH_M} ${VEHICLE_HEIGHT_M}"/></geometry>
-      <material name="cart_white"><color rgba="1.0 1.0 1.0 1.0"/></material>
-    </visual>
-    <collision>
-      <origin xyz="0 0 ${VEHICLE_HEIGHT_M / 2}" rpy="0 0 0"/>
-      <geometry><box size="${VEHICLE_LENGTH_M} ${VEHICLE_WIDTH_M} ${VEHICLE_HEIGHT_M}"/></geometry>
-    </collision>
-    <inertial>
-      <mass value="${VEHICLE_MASS_KG}"/>
-      <origin xyz="0 0 0.5" rpy="0 0 0"/>
-      <inertia ixx="100" iyy="500" izz="500" ixy="0" ixz="0" iyz="0"/>
-    </inertial>
-  </link>
-  <joint name="base_footprint_to_base_link" type="fixed">
-    <parent link="base_footprint"/>
-    <child link="base_link"/>
-    <origin xyz="0 0 0" rpy="0 0 0"/>
-  </joint>
-  -->
-  <!-- ============ Step 3: attach sensor stack to base_link ============ -->
+  <!-- Step 3: attach sensor stack to base_link -->
   <xacro:include filename="$(find gem_sim)/urdf/gem_e4_sensors.urdf.xacro"/>
   <xacro:gem_e4_sensors parent="base_link"/>
